File: kicad/nice_pillz_niceview_v10.kicad_pcb (KiCad board)
At the start: 2 copper layers, 100 x 86 mm, 28 parts, among them J1 Conn_01x13, J2 Conn_01x13, J3 Conn_01x13, J4 Conn_01x13, J5 Conn_01x10, J6 Conn_01x10, J7 Conn_01x13, J8 Conn_01x13, J9 NiceView, M1 MountingHole_6.4mm_M6, M3 MountingHole_4.3mm_M4, M4 MountingHole_4.3mm_M4, U1 nice!nanov2, U2 74HC595

Commit message: PCB v10: switch LED header replaces the external reset terminal
Same two holes at the top of the board, now a 1x02 2.54 mm header for the
LED inside an illuminated power switch: pin 1 (square, "+") is the anode
fed from the switched 3.3 V rail through new series resistor R3 (330R
red/green, 100R blue/white), pin 2 is GND. The 3.3 V feed runs on B.Cu
under COL_5 to a via on the existing rail. The dead RESET branch to the old
terminal is removed; the reset push button keeps its own link to RST.
Silkscreen version v1.1; D1/D2 fab values renamed LED_PWR/LED_BLE.
Project files renamed to v10; JLCPCB Gerbers/drills regenerated.
DRC: 0 unconnected, no new violations except the two library-mismatch
notes for the embedded footprints.

Co-Authored-By: Claude Fable 5.1 <noreply@anthropic.com>
Parts:
- removed Ext. Reset Switch: TerminalBlock_Xinya_XY308-2.54-2P_1x02_P2.54mm_Horizontal, TerminalBlock:TerminalBlock_Xinya_XY308-2.54-2P_1x02_P2.54mm_Horizontal
- added R3: 330R, Resistor_THT:R_Axial_DIN0207_L6.3mm_D2.5mm_P7.62mm_Horizontal, B.Cu at (161.7, 56.0)
- added Switch LED: PinHeader_1x02_P2.54mm_Vertical, Connector_PinHeader_2.54mm:PinHeader_1x02_P2.54mm_Vertical, B.Cu at (161.7, 60.2)
- D1: value LED_CAPS -> LED_PWR
- D2: value LED_NUM -> LED_BLE
Routing:
- net /RESET: track 58.0 -> 33.5 mm
- net +5V: track 55.0 -> 70.4 mm, vias 1 -> 2
- net /SW_LED: track 0.00 -> 4.20 mm
Other:
- board text added: "Nice Pillz View github.com/a10kiloham/nicepillzview v1.1 11 Sep 2026 (built from github/nol00p/nicepillz)"
- board text removed: "Nice Pillz View github.com/a10kiloham/nicepillzview v1.0 29 Aug 2026 (built from github/nol00p/nicepillz)"
